File: mcu.kicad_sch (KiCad schematic)
At the start: 13 parts, among them J2 Conn_2Rows-05Pins, U1 M24C02-RMN, U2 STM32C031C6Tx, Y1 8

Commit message: New crystal
Parts:
- Y1: footprint Crystal:Crystal_SMD_3225-4Pin_3.2x2.5mm -> Crystal:Crystal_SMD_2520-4Pin_2.5x2.0mm
Changed lines of the file:
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@@
 			)
 		)
-		(property "Footprint" "Crystal:Crystal_SMD_3225-4Pin_3.2x2.5mm"
+		(property "Footprint" "Crystal:Crystal_SMD_2520-4Pin_2.5x2.0mm"
 			(at 114.3 44.45 0)
 			(effects
@@
 			)
 		)
-		(property "Datasheet" "~"
+		(property "Datasheet" "https://www.mouser.pl/ProductDetail/Bussmann-Eaton/E2X480081G08?qs=%252BXxaIXUDbq3GNbm8O4NmQg%3D%3D"
 			(at 114.3 44.45 0)
 			(effects
