File: mcu.kicad_sch (KiCad schematic)
At the start: 13 parts, among them J2 Conn_2Rows-05Pins, U1 M24C02-RMN, U2 STM32C031C6Tx, Y1 8

Commit message: 2.1
Connections:
- net LATCH_PIN: no longer names the net of U2.46 (PB7)
- net SPI_MOSI: no longer names the net of U2.44 (PB5)
- net SPI_SCK: no longer names the net of U2.45 (PB6)
Changed lines of the file:
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@@
-		)
-	)
-	(hierarchical_label "LATCH_PIN"
-		(shape input)
-		(at 153.67 99.06 0)
-		(fields_autoplaced yes)
-		(effects
-			(font
-				(size 1.27 1.27)
-			)
-			(justify left)
 		)
 	)
@@
 		)
 	)
-	(hierarchical_label "SPI_MOSI"
-		(shape input)
-		(at 153.67 93.98 0)
-		(fields_autoplaced yes)
-		(effects
-			(font
-				(size 1.27 1.27)
-			)
-			(justify left)
-		)
-	)
 	(hierarchical_label "r_alert_signal"
 		(shape input)
@@
 		(fields_autoplaced yes)
 		(effects
-			(font
-				(size 1.27 1.27)
-			)
-			(justify left)
-		)
-	)
-	(hierarchical_label "SPI_SCK"
-		(shape input)
-		(at 153.67 96.52 0)
-		(fields_autoplaced yes)
-		(effects

Commit message: connections 1.0
Connections:
- net led_pwm_out_3v3 renamed WS2812B_OUT
Changed lines of the file:
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@@
 		)
 	)
-	(hierarchical_label "led_pwm_out_3v3"
+	(hierarchical_label "WS2812B_OUT"
 		(shape input)
 		(at 125.73 58.42 180)
@@
 		)
 		(instances
-			(project ""
+			(project "rpm_meter"
 				(path "/c95b12ac-441d-4f7a-bd6a-c2e5d81eb286/161f8ec5-4d3d-43af-b95a-56d7e596bfdd"
 					(reference "Y1")
@@
 		)
 		(instances
-			(project ""
+			(project "rpm_meter"
 				(path "/c95b12ac-441d-4f7a-bd6a-c2e5d81eb286/161f8ec5-4d3d-43af-b95a-56d7e596bfdd"
 					(reference "U2")
@@
 		)
 		(instances
-			(project ""
+			(project "rpm_meter"
 				(path "/c95b12ac-441d-4f7a-bd6a-c2e5d81eb286/161f8ec5-4d3d-43af-b95a-56d7e596bfdd"
 					(reference "J2")
@@
 		)
 		(instances
-			(project ""
+			(project "rpm_meter"
 				(path "/c95b12ac-441d-4f7a-bd6a-c2e5d81eb286/161f8ec5-4d3d-43af-b95a-56d7e596bfdd"
 					(reference "U1")
@@
 		)
 		(instances
-			(project ""
+			(project "rpm_meter"
 				(path "/c95b12ac-441d-4f7a-bd6a-c2e5d81eb286/161f8ec5-4d3d-43af-b95a-56d7e596bfdd"
 					(reference "#PWR038")
@@
 		)
 		(instances
-			(project ""
+			(project "rpm_meter"
 				(path "/c95b12ac-441d-4f7a-bd6a-c2e5d81eb286/161f8ec5-4d3d-43af-b95a-56d7e596bfdd"
 					(reference "C4")
@@
 		)
 		(instances
-			(project ""
+			(project "rpm_meter"
 				(path "/c95b12ac-441d-4f7a-bd6a-c2e5d81eb286/161f8ec5-4d3d-43af-b95a-56d7e596bfdd"
 					(reference "#PWR040")
