File: rpm_meter.kicad_sch (KiCad schematic)
At the start: 16 parts, among them J1 Conn_01x01_Socket, J3 Conn_01x01_Socket, J4 Conn_01x01_Socket, J5 Conn_01x01_Socket, J6 Conn_01x01_Socket, J7 Conn_01x01_Socket, SW1 RotaryEncoder_Switch_MP

Commit message: USB footprints
Other:
- added sheet usb (usb.kicad_sch)
- sheet mcu ports: added none; removed LATCH_PIN, SPI_MOSI, SPI_SCK
Changed lines of the file:
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@@
+	(wire
+		(pts
+			(xy 71.12 40.64) (xy 80.01 40.64)
+		)
+		(stroke
+			(width 0)
+			(type default)
+		)
+	)
 	(wire
 		(pts
@@
 			)
 		)
-		(pin "SPI_MOSI" input
-			(at 80.01 62.23 180)
-			(effects
-				(font
-					(size 1.27 1.27)
-				)
-				(justify left)
-			)
-		)
-		(pin "SPI_SCK" input
-			(at 80.01 64.77 180)
-			(effects
-				(font
-					(size 1.27 1.27)
-				)
-				(justify left)
-			)
-		)
-		(pin "LATCH_PIN" input
-			(at 80.01 67.31 180)
-			(effects
-				(font
-					(size 1.27 1.27)
-				)
-				(justify left)
-			)
-		)
 		(pin "ENCODER_BTN" input
 			(at 120.65 111.76 0)
@@
 	)
 	(sheet
-		(at 49.53 62.23)
+		(at 55.88 38.1)
 		(size 15.24 5.08)
 		(fields_autoplaced yes)
@@
 		)
 		(property "Sheetname" "Leds"
-			(at 49.53 61.5184 0)
+			(at 55.88 37.3884 0)
 			(effects
 				(font
@@
 		)
 		(property "Sheetfile" "leds.kicad_sch"
-			(at 49.53 67.8946 0)
+			(at 55.88 43.7646 0)
 			(effects
 				(font
@@
 				)
 				(justify left top)
+				(hide yes)
 			)
 		)
 		(pin "WS2812B_IN" input
-			(at 64.77 64.77 0)
+			(at 71.12 40.64 0)
 			(effects
 				(font
@@
 				)
 			)
+		)
+	)
+	(sheet
+		(at 22.86 101.6)
+		(size 31.75 10.16)
+		(fields_autoplaced yes)
+		(stroke
+			(width 0.1524)
+			(type solid)
+		)
+		(fill
+			(color 0 0 0 0.0000)
+		)
+		(property "Sheetname" "usb"
+			(at 22.86 100.8884 0)
+			(effects
+				(font
+					(size 1.27 1.27)
+				)
+				(justify left bottom)
+			)
+		)
+		(property "Sheetfile" "usb.kicad_sch"
+			(at 22.86 112.3446 0)
+			(effects
+				(font
+					(size 1.27 1.27)
+				)
+				(justify left top)
+			)
+		)
+		(instances
+			(project "rpm_meter"
+				(path "/c95b12ac-441d-4f7a-bd6a-c2e5d81eb286"
+					(page "9")
+				)
+			)
