File: rpm_meter.kicad_sch (KiCad schematic)
At the start: 16 parts, among them J1 Conn_01x01_Socket, J3 Conn_01x01_Socket, J4 Conn_01x01_Socket, J5 Conn_01x01_Socket, J6 Conn_01x01_Socket, J7 Conn_01x01_Socket, SW1 RotaryEncoder_Switch_MP

Commit message: 2.1
Other:
- sheet mcu ports: added none; removed LATCH_PIN, SPI_MOSI, SPI_SCK
Changed lines of the file:
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@@
+	(wire
+		(pts
+			(xy 64.77 64.77) (xy 80.01 64.77)
+		)
+		(stroke
+			(width 0)
+			(type default)
+		)
+	)
 	(wire
 		(pts
@@
 		)
 		(pin "led_pwm_out_3v3" input
-			(at 80.01 40.64 180)
+			(at 80.01 64.77 180)
 			(effects
 				(font
@@
 			)
 		)
-		(pin "SPI_MOSI" input
-			(at 80.01 62.23 180)
-			(effects
-				(font
-					(size 1.27 1.27)
-				)
-				(justify left)
-			)
-		)
-		(pin "SPI_SCK" input
-			(at 80.01 64.77 180)
-			(effects
-				(font
-					(size 1.27 1.27)
-				)
-				(justify left)
-			)
-		)
-		(pin "LATCH_PIN" input
-			(at 80.01 67.31 180)
-			(effects
-				(font
-					(size 1.27 1.27)
-				)
-				(justify left)
-			)
-		)

Commit message: connections 1.0
Other:
- sheet mcu ports: added WS2812B_OUT; removed led_pwm_out_3v3
Changed lines of the file:
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@@
 		)
 		(instances
-			(project ""
+			(project "rpm_meter"
 				(path "/c95b12ac-441d-4f7a-bd6a-c2e5d81eb286"
 					(reference "J1")
@@
 		)
 		(instances
-			(project ""
+			(project "rpm_meter"
 				(path "/c95b12ac-441d-4f7a-bd6a-c2e5d81eb286"
 					(reference "#PWR028")
@@
 		)
 		(instances
-			(project ""
+			(project "rpm_meter"
 				(path "/c95b12ac-441d-4f7a-bd6a-c2e5d81eb286"
 					(reference "SW1")
@@
 			)
 		)
-		(pin "led_pwm_out_3v3" input
-			(at 80.01 64.77 180)
-			(effects
-				(font
-					(size 1.27 1.27)
-				)
-				(justify left)
-			)
-		)
 		(pin "rpm_signal_mcu" input
 			(at 120.65 43.18 0)
@@
 			)
 		)
+		(pin "WS2812B_OUT" input
+			(at 80.01 64.77 180)
+			(effects
+				(font
+					(size 1.27 1.27)
+				)
+				(justify left)
+			)
+		)
