File: usb.kicad_sch (KiCad schematic)
At the start: 2 parts, among them IC2 ISO6521FREUR, U5 FT231XQ

Commit message: New placement
Parts:
- added J8: UJ20-C-V-C-1-SMT-TR, Library_local:UJ20CVC1SMTTR, symbol local_library:UJ20-C-V-C-1-SMT-TR
Changed lines of the file:
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@@
+		)
+	)
+	(symbol
+		(lib_id "local_library:UJ20-C-V-C-1-SMT-TR")
+		(at 207.01 99.06 0)
+		(unit 1)
+		(exclude_from_sim no)
+		(in_bom yes)
+		(on_board yes)
+		(dnp no)
+		(fields_autoplaced yes)
+		(property "Reference" "J8"
+			(at 223.52 91.44 0)
+			(effects
+				(font
+					(size 1.27 1.27)
+				)
+			)
+		)
+		(property "Value" "UJ20-C-V-C-1-SMT-TR"
+			(at 223.52 93.98 0)
+			(effects
+				(font
+					(size 1.27 1.27)
+				)
+			)
+		)
+		(property "Footprint" "Library_local:UJ20CVC1SMTTR"
+			(at 236.22 193.98 0)
+			(effects
+				(font
+					(size 1.27 1.27)
+				)
+				(justify left top)
+				(hide yes)
+			)
+		)
+		(property "Datasheet" "https://www.sameskydevices.com/product/resource/uj20-c-v-c-1-smt-tr.pdf"
+			(at 236.22 293.98 0)
+			(effects
+				(font
+					(size 1.27 1.27)
+				)
+				(justify left top)
+				(hide yes)
+			)
+		)
+		(property "Description" "USB Connectors USB Jack 2.0, Type-C, Vertical, Copper Alloy, Surface Mount, 6.5H, T&R"
+			(at 207.01 99.06 0)
+			(effects
+				(font
+					(size 1.27 1.27)
+				)
+				(hide yes)
+			)
+		)
+		(property "Height" "6.65"
+			(at 236.22 493.98 0)
+			(effects
+				(font
+					(size 1.27 1.27)
+				)
+				(justify left top)
+				(hide yes)
+			)
+		)
+		(property "Mouser Part Number" "179-UJ20CVC1SMTTR"
+			(at 236.22 593.98 0)
+			(effects
+				(font
+					(size 1.27 1.27)
+				)
+				(justify left top)
+				(hide yes)
+			)
+		)
+		(property "Mouser Price/Stock" "https://www.mouser.co.uk/ProductDetail/Same-Sky/UJ20-C-V-C-1-SMT-TR?qs=i8QVZAFTkqRSXXSHLSIhtw%3D%3D"
+			(at 236.22 693.98 0)
+			(effects
+				(font
+					(size 1.27 1.27)
+				)
+				(justify left top)
+				(hide yes)
+			)
+		)
+		(property "Manufacturer_Name" "Same Sky"
+			(at 236.22 793.98 0)
+			(effects
+				(font
+					(size 1.27 1.27)
+				)
+				(justify left top)
+				(hide yes)
+			)
+		)
+		(property "Manufacturer_Part_Number" "UJ20-C-V-C-1-SMT-TR"
+			(at 236.22 893.98 0)
+			(effects
+				(font
+					(size 1.27 1.27)
+				)
+				(justify left top)
+				(hide yes)
+			)
+		)
+		(pin "A5"
+		)
+		(pin "A12"
+		)
+		(pin "4"
+		)
+		(pin "A1"
+		)
+		(pin "A8"
+		)
+		(pin "A9"
+		)
+		(pin "1"
+		)
+		(pin "A4"
+		)
+		(pin "B9"
+		)
+		(pin "A7"
+		)
+		(pin "B4"
+		)
+		(pin "2"
+		)
+		(pin "B1"
+		)
+		(pin "B7"
+		)
+		(pin "B12"
+		)
+		(pin "B5"
+		)
+		(pin "A6"
+		)
+		(pin "B8"
+		)
+		(pin "B6"
+		)
+		(pin "3"
+		)
+		(instances
+			(project ""
+				(path "/c95b12ac-441d-4f7a-bd6a-c2e5d81eb286/af3bada4-4de8-405e-b49e-8c6e58262e3d"
+					(reference "J8")
+					(unit 1)
+				)
+			)
 		)
 	)
